Commit message: Test Gripper Down

File: gripper/finger.urdf.xacro (robot description, xacro)
@@ -37,5 +37,5 @@
         <origin rpy="0 0 0" xyz="0 0 0"/>
         <geometry>
-          <mesh filename="package://mygripper/meshes/Link0.stl" scale="${scale} ${scale} ${scale}"/>
+          <mesh filename="package://trimod_gripper/meshes/Link0.stl" scale="${scale} ${scale} ${scale}"/>
         </geometry>
       </visual>
@@ -43,6 +43,7 @@
         <origin rpy="0 0 0" xyz="0 0 0"/>
         <geometry>
-          <mesh filename="package://mygripper/meshes/Link0_convex.stl" scale="${scale} ${scale} ${scale}"/>
+          <mesh filename="package://trimod_gripper/meshes/Link0_convex.stl" scale="${scale} ${scale} ${scale}"/>
         </geometry>
+        <contact_coefficients mu="10.0" kp="100000.0" kd="100000.0" />
       </collision>
       <inertial>
@@ -56,5 +57,5 @@
         <origin rpy="0 0 0" xyz="0 0 0"/>
         <geometry>
-          <mesh filename="package://mygripper/meshes/Link1.stl" scale="${scale} ${scale} ${scale}"/>
+          <mesh filename="package://trimod_gripper/meshes/Link1.stl" scale="${scale} ${scale} ${scale}"/>
         </geometry>
         <material name="blue">
@@ -65,6 +66,7 @@
         <origin rpy="0 0 0" xyz="0 0 0"/>
         <geometry>
-          <mesh filename="package://mygripper/meshes/Link1_convex.stl" scale="${scale} ${scale} ${scale}"/>
+          <mesh filename="package://trimod_gripper/meshes/Link1_convex.stl" scale="${scale} ${scale} ${scale}"/>
         </geometry>
+        <contact_coefficients mu="10.0" kp="100000.0" kd="100000.0" />
       </collision>
       <inertial>
@@ -78,5 +80,5 @@
         <origin rpy="0 0 0" xyz="0 0 0"/>
         <geometry>
-          <mesh filename="package://mygripper/meshes/Link2.stl" scale="${scale} ${scale} ${scale}"/>
+          <mesh filename="package://trimod_gripper/meshes/Link2.stl" scale="${scale} ${scale} ${scale}"/>
         </geometry>
         <material name="blue">
@@ -87,6 +89,7 @@
         <origin rpy="0 0 0" xyz="0 0 0"/>
         <geometry>
-          <mesh filename="package://mygripper/meshes/Link2_convex.stl" scale="${scale} ${scale} ${scale}"/>
+          <mesh filename="package://trimod_gripper/meshes/Link2_convex.stl" scale="${scale} ${scale} ${scale}"/>
         </geometry>
+        <contact_coefficients mu="10.0" kp="100000.0" kd="100000.0" />
       </collision>
       <inertial>
@@ -96,4 +99,10 @@
       </inertial>
     </link>
+      <gazebo reference="${name}_link2">
+          <mu1>10.0</mu1>
+          <mu2>10.0</mu2>
+          <kp>10000000.0</kp>
+          <kd>10000000.0</kd>
+      </gazebo>
 <!-- JOINTS -->
     <joint name="${name}_joint_base" type="fixed">

File: gripper/single_trimod.urdf.xacro (robot description, xacro)
@@ -1,8 +1,8 @@
 <?xml version="1.0"?>
 <robot name="trimod" xmlns:xacro="http://www.ros.org/wiki/xacro">
-  <xacro:include filename="$(find mygripper)/gripper/trimod.urdf.xacro"/>
+  <xacro:include filename="$(find trimod_gripper)/gripper/trimod.urdf.xacro"/>
   <link name="world" />
   <trimod name="trimod" parent="world">
-    <origin rpy="0 0 0" xyz="0 0 0.2"/>
+    <origin rpy="${M_PI} 0 0" xyz="0 0 0.4"/>
   </trimod>
 </robot>

File: gripper/trimod.urdf.xacro (robot description, xacro)
@@ -1,6 +1,6 @@
 <?xml version="1.0"?>
 <robot xmlns:xacro="http://www.ros.org/wiki/xacro">
-  <xacro:include filename="$(find mygripper)/gripper/utils.urdf.xacro"/>
-  <xacro:include filename="$(find mygripper)/gripper/finger.urdf.xacro"/>
+  <xacro:include filename="$(find trimod_gripper)/gripper/utils.urdf.xacro"/>
+  <xacro:include filename="$(find trimod_gripper)/gripper/finger.urdf.xacro"/>
   <xacro:property name="gripper_r" value="${0.02}"/>
   <xacro:property name="gripper_d" value="${gripper_r*1.4641}"/>

Commit message: new features

File: gripper/finger.urdf.xacro (robot description, xacro)
@@ -1,4 +1,4 @@
 <?xml version="1.0"?>
-<robot xmlns:xacro="http://www.ros.org/wiki/xacro">
+<robot name="trimod" xmlns:xacro="http://www.ros.org/wiki/xacro">
   <xacro:property name="scale" value="0.1"/>
   <xacro:property name="fingerDepth" value="0.2"/>
@@ -9,4 +9,5 @@
   <xacro:property name="effort" value="10"/>
   <xacro:property name="interface" value="PositionJointInterface"/>
+  <xacro:property name="mass" value="0.2"/>
   <!--<xacro:property name="interface" value="EffortJointInterface"/>-->
   <macro name="finger" params="name parent *origin">
@@ -29,6 +30,6 @@
       <inertial>
         <origin rpy="0 0 0" xyz="0 0 0"/>
-        <mass value="1"/>
-        <box_inertia m="1" x="0.01" y="0.01" z="0.01"/>
+        <mass value="${mass/4}"/>
+        <box_inertia m="${mass/4}" x="0.01" y="0.01" z="0.01"/>
       </inertial>
     </link>
@@ -49,6 +50,6 @@
       <inertial>
         <origin rpy="0 0 0" xyz="${fingerDepth*scale*0.5} 0.000000 ${fingerDepth*scale*0.5}"/>
-        <mass value="1000"/>
-        <box_inertia m="1000" x="${link0r*scale}" y="${fingerDepth*scale}" z="${0.2*scale}"/>
+        <mass value="${mass/4}"/>
+        <box_inertia m="${mass/4}" x="${link0r*scale}" y="${fingerDepth*scale}" z="${0.2*scale}"/>
       </inertial>
     </link>
@@ -72,6 +73,6 @@
       <inertial>
         <origin rpy="0 0 0" xyz="${link1a*scale*0.5} 0.000000 0.000000"/>
-        <mass value="1"/>
-        <box_inertia m="1" x="${link1a*scale}" y="${fingerDepth*scale}" z="${fingerDepth*scale}"/>
+        <mass value="${mass/4}"/>
+        <box_inertia m="${mass/4}" x="${link1a*scale}" y="${fingerDepth*scale}" z="${fingerDepth*scale}"/>
       </inertial>
     </link>
@@ -95,6 +96,6 @@
       <inertial>
         <origin rpy="0 0 0" xyz="${link2a*scale*0.5} 0.000000 0.000000"/>
-        <mass value="10"/>
-        <box_inertia m="10" x="${link2a*scale}" y="${fingerDepth*scale}" z="${fingerDepth*scale}"/>
+        <mass value="${mass/4}"/>
+        <box_inertia m="${mass/4}" x="${link2a*scale}" y="${fingerDepth*scale}" z="${fingerDepth*scale}"/>
       </inertial>
     </link>
@@ -122,5 +123,5 @@
       <parent link="${name}_link0"/>
       <child link="${name}_link1"/>
-      <origin rpy="${pi/2} -${pi/2} 0" xyz="${link0r*scale} 0 ${link0h*scale}"/>
+      <origin rpy="${M_PI/2} -${M_PI/2} 0" xyz="${link0r*scale} 0 ${link0h*scale}"/>
       <axis xyz="0 0 1"/>
       <limit effort="${effort}" lower="${-90 * M_PI / 180}" upper="${50 * M_PI / 180}" velocity="100"/>

File: gripper/trimod.urdf.xacro (robot description, xacro)
@@ -1,4 +1,4 @@
 <?xml version="1.0"?>
-<robot xmlns:xacro="http://www.ros.org/wiki/xacro">
+<robot name="trimod" xmlns:xacro="http://www.ros.org/wiki/xacro">
   <xacro:include filename="$(find trimod_gripper)/gripper/utils.urdf.xacro"/>
   <xacro:include filename="$(find trimod_gripper)/gripper/finger.urdf.xacro"/>
@@ -8,4 +8,5 @@
   <xacro:property name="gripper_a" value="${0.5774*(gripper_d*0.5+gripper_r)}"/>
   <xacro:property name="gripper_b" value="${(gripper_d*0.5+gripper_r)/0.8660}"/>
+  <xacro:property name="gripper_mass" value="0.2"/>
   <macro name="trimod" params="name parent *origin">
     <link name="${name}_base">
@@ -27,6 +28,6 @@
       <inertial>
         <origin rpy="${M_PI/2} 0 0" xyz="0 0 0"/>
-        <mass value="1000000"/>
-        <cylinder_inertia length="0.01" mass="1000000" radius="0.04"/>
+        <mass value="${gripper_mass}"/>
+        <cylinder_inertia length="0.01" mass="${gripper_mass}" radius="0.04"/>
       </inertial>
     </link>
@@ -45,9 +46,14 @@
       <origin rpy="0 0 0" xyz="${gripper_b} 0 0.0"/>
     </finger>
+    <gazebo>
+      <plugin filename="libgazebo_ros_control.so" name="trimod_gazebo_ros_control">
+        <robotNamespace>/trimod</robotNamespace>
+      </plugin>
+    </gazebo>
+    <!--<gazebo>
+        <plugin name="${name}_lwr_hw_sim" filename="liblwr_hw_gazebo_plugin.so">
+            <robotNamespace>${name}</robotNamespace>
+        </plugin>
+    </gazebo>-->
   </macro>
-  <gazebo>
-    <plugin filename="libgazebo_ros_control.so" name="gazebo_ros_control">
-      <robotNamespace>/trimod</robotNamespace>
-    </plugin>
-  </gazebo>
 </robot>

File: gripper/utils.urdf.xacro (robot description, xacro)
@@ -1,5 +1,4 @@
 <?xml version="1.0"?>
-<robot name="trimod" xmlns:xacro="http://www.ros.org/wiki/xacro">
-  <xacro:property name="pi" value="3.1415926535897931"/>
+<robot  xmlns:xacro="http://www.ros.org/wiki/xacro">
   <xacro:property name="M_PI" value="3.1415926535897931"/>
   <xacro:macro name="cuboid_inertia" params="width height length mass">
@@ -16,6 +15,6 @@
              ixy="0" iyz="0" ixz="0"/>
   </xacro:macro>
-  <macro name="box_inertia" params="m x:=${x} y z">
+  <xacro:macro name="box_inertia" params="m x:=${x} y z">
     <inertia ixx="${m*(y*y+z*z)/12}" ixy="0" ixz="0" iyy="${m*(x*x+z*z)/12}" iyz="0" izz="${m*(x*x+z*z)/12}"/>
-  </macro>
+  </xacro:macro>
 </robot>

Commit message: Grasp Test

File: gripper/finger.urdf.xacro (robot description, xacro)
@@ -7,8 +7,10 @@
   <xacro:property name="link1a" value="0.6"/>
   <xacro:property name="link2a" value="0.4"/>
-  <xacro:property name="effort" value="10"/>
-  <xacro:property name="interface" value="PositionJointInterface"/>
-  <xacro:property name="mass" value="0.2"/>
-  <!--<xacro:property name="interface" value="EffortJointInterface"/>-->
+  <xacro:property name="effort" value="50"/>
+  <xacro:property name="jdamping" value="0.03"/>
+  <xacro:property name="jfriction" value="3.0"/>
+<!--<xacro:property name="interface" value="PositionJointInterface"/>-->
+  <xacro:property name="interface" value="EffortJointInterface"/>
+  <xacro:property name="mass" value="1"/>
   <macro name="finger" params="name parent *origin">
     <link name="${name}_base">
@@ -46,5 +48,5 @@
           <mesh filename="package://trimod_gripper/meshes/Link0_convex.stl" scale="${scale} ${scale} ${scale}"/>
         </geometry>
-        <contact_coefficients mu="10.0" kp="100000.0" kd="100000.0" />
+        <contact_coefficients kd="100000.0" kp="100000.0" mu="10.0"/>
       </collision>
       <inertial>
@@ -69,5 +71,5 @@
           <mesh filename="package://trimod_gripper/meshes/Link1_convex.stl" scale="${scale} ${scale} ${scale}"/>
         </geometry>
-        <contact_coefficients mu="10.0" kp="100000.0" kd="100000.0" />
+        <contact_coefficients kd="100000.0" kp="100000.0" mu="10.0"/>
       </collision>
       <inertial>
@@ -87,11 +89,5 @@
         </material>
       </visual>
-      <collision>
-        <origin rpy="0 0 0" xyz="0 0 0"/>
-        <geometry>
-          <mesh filename="package://trimod_gripper/meshes/Link2_convex.stl" scale="${scale} ${scale} ${scale}"/>
-        </geometry>
-        <contact_coefficients mu="10.0" kp="100000.0" kd="100000.0" />
-      </collision>
+      <collision_sphere radius="${link0r*scale*0.5}" rpy="0 0 0" xyz="${link2a*scale} 0 0"/>
       <inertial>
         <origin rpy="0 0 0" xyz="${link2a*scale*0.5} 0.000000 0.000000"/>
@@ -100,12 +96,31 @@
       </inertial>
     </link>
-      <gazebo reference="${name}_link2">
-          <mu1>300000.0</mu1>
-          <mu2>300000.0</mu2>
-          <kp>10000000.0</kp>
-          <kd>10000000.0</kd>
-          <slip1>1000.0</slip1>
-          <slip2>1000.0</slip2>
-      </gazebo>
+    <gazebo reference="${name}_link2">
+      <kp>10000000000</kp>
+      <kd>0.01</kd>
+      <mu1>Inf</mu1>
+      <mu2>Inf</mu2>
+      <gripper name="${name}_gripper">
+        <grasp_check>
+          <attach_steps>5</attach_steps>
+          <detach_steps>10</detach_steps>
+        </grasp_check>
+        <gripper_link>${name}_link2</gripper_link>
+        <palm_link>${name}_link1</palm_link>
+      </gripper>
+      <sensor name="${name}_fixed_jaw_contact_sensor" type="contact">
+        <always_on>true</always_on>
+        <update_rate>20</update_rate>
+        <contact>
+<!-- When using ROS Indigo and Gazebo 2.2.3, the name specified here
+               must be <link name>_collision. -->
+          <collision>${name}_link2_collision</collision>
+        </contact>
+        <plugin filename="libgazebo_ros_bumper.so" name="${name}_fixed_jaw_bumper">
+          <bumperTopicName>${name}_sensor_state</bumperTopicName>
+          <frameName>${name}_link2</frameName>
+        </plugin>
+      </sensor>
+    </gazebo>
 <!-- JOINTS -->
     <joint name="${name}_joint_base" type="fixed">
@@ -120,5 +135,5 @@
       <axis xyz="0 0 1"/>
       <limit effort="${effort}" lower="${-90 * M_PI / 180}" upper="${90 * M_PI / 180}" velocity="100"/>
-      <dynamics damping="1.0" friction="10.0"/>
+      <dynamics damping="${jdamping}" friction="${jfriction}"/>
     </joint>
     <joint name="${name}_joint_proximal" type="revolute">
@@ -128,5 +143,5 @@
       <axis xyz="0 0 1"/>
       <limit effort="${effort}" lower="${-90 * M_PI / 180}" upper="${50 * M_PI / 180}" velocity="100"/>
-      <dynamics damping="1.0" friction="10.0"/>
+      <dynamics damping="${jdamping}" friction="${jfriction}"/>
     </joint>
     <joint name="${name}_joint_distal" type="revolute">
@@ -136,5 +151,5 @@
       <axis xyz="0 0 1"/>
       <limit effort="${effort}" lower="${-90 * M_PI / 180}" upper="${90 * M_PI / 180}" velocity="100"/>
-      <dynamics damping="1.0" friction="10.0"/>
+      <dynamics damping="${jdamping}" friction="${jfriction}"/>
     </joint>
 <!-- TRANSMISSIONS -->

File: gripper/utils.urdf.xacro (robot description, xacro)
@@ -18,3 +18,12 @@
     <inertia ixx="${m*(y*y+z*z)/12}" ixy="0" ixz="0" iyy="${m*(x*x+z*z)/12}" iyz="0" izz="${m*(x*x+z*z)/12}"/>
   </xacro:macro>
+  <xacro:macro name="collision_sphere" params="radius xyz rpy">
+    <collision>
+      <origin rpy="${rpy}" xyz="${xyz}"/>
+      <geometry>
+        <sphere radius="${radius}"/>
+      </geometry>
+      <contact_coefficients mu="100000000.0" mu2="100000000.0" kp="100000.0" kd="100000.0" />
+    </collision>
+  </xacro:macro>
 </robot>

Commit message: Added Gripper Tag

File: gripper/finger.urdf.xacro (robot description, xacro)
@@ -101,18 +101,9 @@
       <mu1>Inf</mu1>
       <mu2>Inf</mu2>
-      <gripper name="${name}_gripper">
-        <grasp_check>
-          <attach_steps>5</attach_steps>
-          <detach_steps>10</detach_steps>
-        </grasp_check>
-        <gripper_link>${name}_link2</gripper_link>
-        <palm_link>${name}_link1</palm_link>
-      </gripper>
+      <!--
       <sensor name="${name}_fixed_jaw_contact_sensor" type="contact">
         <always_on>true</always_on>
         <update_rate>20</update_rate>
         <contact>
-<!-- When using ROS Indigo and Gazebo 2.2.3, the name specified here
-               must be <link name>_collision. -->
           <collision>${name}_link2_collision</collision>
         </contact>
@@ -122,4 +113,5 @@
         </plugin>
       </sensor>
+    -->
     </gazebo>
 <!-- JOINTS -->

File: gripper/trimod.urdf.xacro (robot description, xacro)
@@ -51,4 +51,16 @@
       </plugin>
     </gazebo>
+    <gazebo>
+      <gripper name="${name}_gripper">
+        <grasp_check>
+          <attach_steps>5</attach_steps>
+          <detach_steps>10</detach_steps>
+        </grasp_check>
+        <gripper_link>${name}_finger_left_link2</gripper_link>
+        <gripper_link>${name}_finger_right_link2</gripper_link>
+        <gripper_link>${name}_finger_center_link2</gripper_link>
+        <palm_link>${name}_base</palm_link>
+      </gripper>
+    </gazebo>
     <!--<gazebo>
         <plugin name="${name}_lwr_hw_sim" filename="liblwr_hw_gazebo_plugin.so">

Commit message: chinese test

File: gripper/finger.urdf.xacro (robot description, xacro)
@@ -101,5 +101,5 @@
       <mu1>Inf</mu1>
       <mu2>Inf</mu2>
-      <!--
+<!--
       <sensor name="${name}_fixed_jaw_contact_sensor" type="contact">
         <always_on>true</always_on>

File: gripper/trimod.urdf.xacro (robot description, xacro)
@@ -12,16 +12,13 @@
     <link name="${name}_base">
       <visual>
-        <origin rpy="0 0 0" xyz="0 0 0"/>
+        <origin rpy="0 0 0" xyz="0 0 -0.02"/>
         <geometry>
-          <cylinder length="0.01" radius="0.04"/>
+          <cylinder length="0.04" radius="0.04"/>
         </geometry>
-        <material name="blue">
-          <color rgba="0 0 .8 1"/>
-        </material>
       </visual>
       <collision>
-        <origin rpy="0 0 0" xyz="0 0 0"/>
+        <origin rpy="0 0 0" xyz="0 0 -0.02"/>
         <geometry>
-          <cylinder length="0.01" radius="0.04"/>
+          <cylinder length="0.04" radius="0.04"/>
         </geometry>
       </collision>
@@ -64,4 +61,16 @@
       </gripper>
     </gazebo>
+    <gazebo reference="${name}_finger_left">
+      <material>Gazebo/Red</material>
+    </gazebo>
+    <gazebo reference="${name}_finger_right">
+      <material>Gazebo/Red</material>
+    </gazebo>
+    <gazebo reference="${name}_finger_center">
+      <material>Gazebo/Red</material>
+    </gazebo>
+    <gazebo reference="${name}_base">
+      <material>Gazebo/Grey</material>
+    </gazebo>
     <!--<gazebo>
         <plugin name="${name}_lwr_hw_sim" filename="liblwr_hw_gazebo_plugin.so">

File: gripper/utils.urdf.xacro (robot description, xacro)
@@ -27,3 +27,9 @@
     </collision>
   </xacro:macro>
+  <material name="pino">
+     <color rgba="${158/255} ${22/255} ${22/255} 1.0"/>
+  </material>
+  <material name="gred">
+     <color rgba="${0/255} ${175/255} ${175/255} 1.0"/>
+  </material>
 </robot>
